File: PCB_project/IO.kicad_sch (KiCad schematic)
At the start: 12 parts, among them Q1 AO3400A

Commit message: Almost ready version. Require more GND vias etc
Parts:
- added R44: 1k, Resistor_SMD:R_0402_1005Metric, symbol Device:R
- LS1: value CBT-09427-SMT -> GMD0955YB-3V2700
Connections:
- net +3V3: now also R44.1
- net at D14.2 (A), LS1.2 (-), Q1.3 (D): now also R44.2
Other:
- moved on the sheet: D14
Changed lines of the file:
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@@
+	)
+	(junction
+		(at 242.57 88.9)
+		(diameter 0)
+		(color 0 0 0 0)
 	)
 	(junction
@@
 	)
 	(junction
+		(at 242.57 76.2)
+		(diameter 0)
+		(color 0 0 0 0)
+	)
+	(junction
 		(at 251.46 101.6)
 		(diameter 0)
@@
 	(wire
 		(pts
-			(xy 251.46 74.93) (xy 251.46 76.2)
+			(xy 242.57 88.9) (xy 251.46 88.9)
 		)
 		(stroke
@@
 	(wire
 		(pts
-			(xy 251.46 76.2) (xy 251.46 77.47)
+			(xy 251.46 74.93) (xy 251.46 76.2)
 		)
 		(stroke
@@
 	(wire
 		(pts
-			(xy 251.46 87.63) (xy 251.46 88.9)
+			(xy 251.46 76.2) (xy 251.46 77.47)
 		)
 		(stroke
@@
 	(wire
 		(pts
-			(xy 251.46 88.9) (xy 251.46 90.17)
+			(xy 242.57 86.36) (xy 242.57 88.9)
 		)
 		(stroke
@@
 	(wire
 		(pts
-			(xy 121.92 77.47) (xy 139.7 77.47)
+			(xy 251.46 87.63) (xy 251.46 88.9)
 		)
 		(stroke
@@
 	(wire
 		(pts
-			(xy 245.11 86.36) (xy 245.11 88.9)
+			(xy 251.46 88.9) (xy 251.46 90.17)
 		)
 		(stroke
@@
 	(wire
 		(pts
-			(xy 74.93 77.47) (xy 77.47 77.47)
+			(xy 121.92 77.47) (xy 139.7 77.47)
 		)
 		(stroke
@@
 	(wire
 		(pts
-			(xy 154.94 77.47) (xy 170.18 77.47)
+			(xy 236.22 86.36) (xy 236.22 88.9)
 		)
 		(stroke
@@
 	(wire
 		(pts
-			(xy 245.11 88.9) (xy 251.46 88.9)
+			(xy 74.93 77.47) (xy 77.47 77.47)
 		)
 		(stroke
@@
 	(wire
 		(pts
-			(xy 251.46 101.6) (xy 251.46 100.33)
+			(xy 242.57 76.2) (xy 251.46 76.2)
 		)
 		(stroke
@@
 	(wire
 		(pts
-			(xy 245.11 78.74) (xy 245.11 76.2)
+			(xy 154.94 77.47) (xy 170.18 77.47)
 		)
 		(stroke
@@
 	(wire
 		(pts
-			(xy 243.84 95.25) (xy 243.84 101.6)
+			(xy 236.22 88.9) (xy 242.57 88.9)
 		)
 		(stroke
@@
 	(wire
 		(pts
-			(xy 240.03 95.25) (xy 243.84 95.25)
+			(xy 251.46 101.6) (xy 251.46 100.33)
 		)
 		(stroke
@@
 	(wire
 		(pts
-			(xy 92.71 77.47) (xy 106.68 77.47)
+			(xy 236.22 78.74) (xy 236.22 76.2)
 		)
 		(stroke
@@
 	(wire
 		(pts
-			(xy 245.11 76.2) (xy 251.46 76.2)
+			(xy 243.84 95.25) (xy 243.84 101.6)
+		)
+		(stroke
+			(width 0)
+			(type default)
+		)
+	)
+	(wire
+		(pts
+			(xy 240.03 95.25) (xy 243.84 95.25)
+		)
+		(stroke
+			(width 0)
+			(type default)
+		)
+	)
+	(wire
+		(pts
+			(xy 92.71 77.47) (xy 106.68 77.47)
+		)
+		(stroke
+			(width 0)
+			(type default)
+		)
+	)
+	(wire
+		(pts
+			(xy 236.22 76.2) (xy 242.57 76.2)
+		)
+		(stroke
+			(width 0)
+			(type default)
+		)
+	)
+	(wire
+		(pts
+			(xy 242.57 76.2) (xy 242.57 78.74)
 		)
 		(stroke
@@
 		(fields_autoplaced yes)
 		(property "Reference" "LS1"
-			(at 255.27 80.7376 0)
+			(at 255.27 81.1542 0)
 			(show_name no)
 			(do_not_autoplace no)
@@
 			)
 		)
-		(property "Value" "CBT-09427-SMT"
-			(at 255.27 83.2776 0)
+		(property "Value" "GMD0955YB-3V2700"
+			(at 255.27 83.6942 0)
 			(show_name no)
 			(do_not_autoplace no)
@@
 	(symbol
 		(lib_id "Diode:1N4148")
-		(at 245.11 82.55 270)
+		(at 236.22 82.55 270)
 		(unit 1)
 		(body_style 1)
@@
 		(dnp no)
 		(property "Reference" "D14"
-			(at 234.95 81.28 90)
+			(at 226.06 81.28 90)
 			(show_name no)
 			(do_not_autoplace no)
@@
 		)
 		(property "Value" "B5819W SL"
-			(at 232.41 84.074 90)
+			(at 223.52 84.074 90)
 			(show_name no)
 			(do_not_autoplace no)
@@
 		)
 		(property "Footprint" "Diode_SMD:D_SOD-123"
-			(at 240.665 82.55 0)
+			(at 231.775 82.55 0)
 			(hide yes)
 			(show_name no)
@@
 		)
 		(property "Datasheet" "https://assets.nexperia.com/documents/data-sheet/1N4148_1N4448.pdf"
-			(at 245.11 82.55 0)
-			(hide yes)
-			(show_name no)
-			(do_not_autoplace no)
-			(effects
-				(font
-					(size 1.27 1.27)
-				)
-			)
-		)
-		(property "Description" ""
-			(at 245.11 82.55 0)
+			(at 236.22 82.55 0)
+			(hide yes)
+			(show_name no)
+			(do_not_autoplace no)
+			(effects
+				(font
+					(size 1.27 1.27)
+				)
+			)
+		)
+		(property "Description" ""
+			(at 236.22 82.55 0)
 			(show_name no)
 			(do_not_autoplace no)
@@
 					(unit 1)
 				)
+			)
+		)
+	)
+	(symbol
+		(lib_id "Device:R")
+		(at 242.57 82.55 0)
+		(unit 1)
+		(body_style 1)
+		(exclude_from_sim no)
+		(in_bom yes)
+		(on_board yes)
+		(in_pos_files yes)
+		(dnp no)
+		(property "Reference" "R44"
+			(at 240.03 83.82 90)
+			(show_name no)
+			(do_not_autoplace no)
+			(effects
+				(font
+					(size 1.27 1.27)
+				)
+			)
+		)
+		(property "Value" "1k"
+			(at 245.11 83.82 90)
+			(show_name no)
+			(do_not_autoplace no)
+			(effects
+				(font
+					(size 1.27 1.27)
+				)
+			)
+		)
+		(property "Footprint" "Resistor_SMD:R_0402_1005Metric"
+			(at 240.792 82.55 90)
+			(hide yes)
+			(show_name no)
+			(do_not_autoplace no)
+			(effects
+				(font
+					(size 1.27 1.27)
+				)
+			)
+		)
+		(property "Datasheet" ""
+			(at 242.57 82.55 0)
+			(hide yes)
+			(show_name no)
+			(do_not_autoplace no)
+			(effects
+				(font
+					(size 1.27 1.27)
+				)
+			)
+		)
+		(property "Description" ""
+			(at 242.57 82.55 0)
+			(show_name no)
+			(do_not_autoplace no)
+			(effects
+				(font
+					(size 1.27 1.27)
+				)
+			)
+		)
+		(pin "1"
+		)
+		(pin "2"
+		)
+		(instances
+			(project "kp-ptr"
+				(path "/9538e4ed-27e6-4c37-b989-9859dc0d49e8/68d9bec4-a8fa-482b-99d8-a42578238d37"
+					(reference "R44")
+					(unit 1)
+				)
